Commit message: commit_4

File: urdf/arm_1.urdf (robot description, URDF)
Before this commit: robot arm_1, 4 links, 3 joints
Links:
- added link link_04, mass 0.02; collision cylinder length=0.02 radius=0.02; visual cylinder length=0.02 radius=0.02
Joints:
- added joint joint3: type fixed, parent link_03, child link_04, origin xyz=0 0 -.175 rpy=0 0 0, axis 0 1 0
- joint joint1: limit lower=-1.57 upper=0 effort=1000 velocity=.5 -> lower=0 upper=1.57 effort=1000 velocity=.5; origin xyz=0 0 0 rpy=0 1.57 0 -> xyz=0 0 0 rpy=0 0 0
- joint joint2: origin xyz=0 0 -0.2 rpy=0 -3.14 0 -> xyz=0 0 -0.2 rpy=0 -1.57 0
